Commit message: Added hdl_slam (3D slam)

File: rosbot_description/src/rosbot_description/urdf/rosbot_default.xacro (robot description, xacro)
@@ -2,5 +2,4 @@
 <robot name="rosbot"
   xmlns:xacro="http://www.ros.org/wiki/xacro">
-  <xacro:property name="M_PI" value="3.1415926535897931" />
   <xacro:arg name="robot_namespace" default=""/>
   <xacro:property name="cameraSize" value="0.05"/>
@@ -293,5 +292,5 @@
   </joint>
   <!-- rplidar Laser -->
-  <!-- <link name="laser">
+  <link name="laser">
     <collision>
       <origin xyz="0 0 0.058" rpy="1.5707 0 4.71"/>
@@ -311,50 +310,4 @@
       <inertia ixx="0" ixy="0" ixz="0" iyy="0" iyz="0" izz="0" />
     </inertial>
-  </link> -->
-<!-- Velodyne Link Stuff -->
-  <link name="laser">
-    <collision>
-      <origin xyz="0 0 0.058" rpy="1.5707 0 4.71"/>
-      <geometry>
-        <cylinder radius="0.0516" length="0.0717"/>
-      </geometry>
-    </collision>
-    <visual>
-      <origin xyz="0 0 0.058" rpy="1.5707 0 4.71"/>
-      <geometry>
-        <mesh filename="package://rosbot_description/meshes/VLP16_base_1.dae" scale="0.001 0.001 0.001" />
-      </geometry>
-    </visual>
-    <visual>
-      <origin xyz="0 0 0.058" rpy="1.5707 0 4.71"/>
-      <geometry>
-        <mesh filename="package://rosbot_description/meshes/VLP16_base_2.dae" scale="0.001 0.001 0.001" />
-      </geometry>
-    </visual>
-    <inertial>
-      <mass value="0.83"/>
-      <origin xyz="0 0 0.03585"/>
-      <inertia ixx="${(0.83 * (3.0*0.0516*0.0516 + 0.0717*0.0717)) / 12.0}" ixy="0" ixz="0"
-        iyy="${(0.83 * (3.0*0.0516*0.0516 + 0.0717*0.0717)) / 12.0}" iyz="0"
-        izz="${0.5 * 0.83 * (0.0516*0.0516)}"/>
-    </inertial>
-  </link>
-  <joint name="$laser_base_scan_joint" type="fixed" >
-    <origin xyz="0 0 0.0377" rpy="0 0 0" />
-    <parent link="laser" />
-    <child link="laser_velodyne"/>
-  </joint>
-  <link name="laser_velodyne">
-    <inertial>
-      <mass value="0.01"/>
-      <origin xyz="0 0 0"/>
-      <inertia ixx="1e-7" ixy="0" ixz="0" iyy="1e-7" iyz="0" izz="1e-7"/>
-    </inertial>
-    <visual>
-      <origin xyz="0 0 -0.0377" />
-      <geometry>
-        <mesh filename="package://rosbot_description/meshes/VLP16_scan.dae" scale="0.001 0.001 0.001" />
-      </geometry>
-    </visual>
   </link>
   <joint name="range_fl_joint" type="fixed">
