Commit message: Lidar is now visible on model.

File: rosbot_description/src/rosbot_description/urdf/rosbot.xacro (robot description, xacro)
@@ -286,10 +286,10 @@
   <link name="camera_depth_frame">
   </link>
-  <joint name="rplidar_joint" type="fixed">
+  <!-- <joint name="rplidar_joint" type="fixed">
     <axis xyz="0 1 0" />
     <origin xyz="0.02 0 0" rpy="0 0 3.14"/>
     <parent link="base_link"/>
     <child link="laser"/>
-  </joint>
+  </joint> -->
   <!-- rplidar Laser -->
   <!-- <link name="laser">
@@ -313,5 +313,5 @@
   </link> -->
 <!-- Velodyne Link Stuff -->
-  <link name="laser">
+  <!-- <link name="laser">
     <collision>
       <origin xyz="0 0 0.058" rpy="1.5707 0 4.71"/>
@@ -357,5 +357,10 @@
       </geometry>
     </visual>
-  </link>
+  </link> -->
+<!-- Velodyne Include Stuff -->
+  <xacro:include filename="$(find rosbot_description)/urdf/VLP-16-modified.urdf.xacro"/>
+  <VLP-16 parent="base_link" name="velodyne" topic="/velodyne_points" hz="10" samples="440" gpu="false">
+    <origin xyz="0.025 0 0.055" rpy="0 0 0" />
+  </VLP-16>
   <joint name="range_fl_joint" type="fixed">
     <axis xyz="0 1 0" />
