Commit message: Moved all Velodyne Rosbot files into the central lidar_interface package.

File: lidar_interface/urdf/VLP-16-modified.urdf.xacro (robot description, xacro)
@@ -18,10 +18,10 @@
       <visual>
         <geometry>
-          <mesh filename="package://rosbot_description/meshes/VLP16_base_1.dae" />
+          <mesh filename="package://velodyne_description/meshes/VLP16_base_1.dae" />
         </geometry>
       </visual>
       <visual>
         <geometry>
-          <mesh filename="package://rosbot_description/meshes/VLP16_base_2.dae" />
+          <mesh filename="package://velodyne_description/meshes/VLP16_base_2.dae" />
         </geometry>
       </visual>
@@ -47,5 +47,5 @@
         <origin xyz="0 0 -0.0377" />
         <geometry>
-          <mesh filename="package://rosbot_description/meshes/VLP16_scan.dae" />
+          <mesh filename="package://velodyne_description/meshes/VLP16_scan.dae" />
         </geometry>
       </visual>

File: lidar_interface/urdf/rosbot_velodyne.xacro (robot description, xacro)
@@ -2,9 +2,10 @@
 <robot name="rosbot"
   xmlns:xacro="http://www.ros.org/wiki/xacro">
+  <xacro:property name="M_PI" value="3.1415926535897931" />
   <xacro:arg name="robot_namespace" default=""/>
   <xacro:property name="cameraSize" value="0.05"/>
   <xacro:property name="cameraMass" value="0.1"/>
   <xacro:property name="namespace" value="$(arg robot_namespace)" />
-  <xacro:include filename="$(find rosbot_description)/urdf/rosbot.gazebo" />
+  <xacro:include filename="$(find lidar_interface)/urdf/rosbot_velodyne.gazebo" />
   <xacro:include filename="$(find rosbot_description)/urdf/materials.xacro" />
   <xacro:include filename="$(find rosbot_description)/urdf/macros.xacro" />
@@ -285,12 +286,12 @@
   <link name="camera_depth_frame">
   </link>
-  <joint name="rplidar_joint" type="fixed">
+  <!-- <joint name="rplidar_joint" type="fixed">
     <axis xyz="0 1 0" />
     <origin xyz="0.02 0 0" rpy="0 0 3.14"/>
     <parent link="base_link"/>
     <child link="laser"/>
-  </joint>
+  </joint> -->
   <!-- rplidar Laser -->
-  <link name="laser">
+  <!-- <link name="laser">
     <collision>
       <origin xyz="0 0 0.058" rpy="1.5707 0 4.71"/>
@@ -310,5 +311,10 @@
       <inertia ixx="0" ixy="0" ixz="0" iyy="0" iyz="0" izz="0" />
     </inertial>
-  </link>
+  </link> -->
+<!-- Velodyne LIDAR -->
+  <xacro:include filename="$(find lidar_interface)/urdf/VLP-16-modified.urdf.xacro"/>
+  <VLP-16 parent="base_link" name="velodyne" topic="/velodyne_points" hz="10" samples="440" gpu="false">
+    <origin xyz="0.025 0 0.055" rpy="0 0 0" />
+  </VLP-16>
   <joint name="range_fl_joint" type="fixed">
     <axis xyz="0 1 0" />

File: rosbot_description/src/rosbot_description/urdf/rosbot.xacro (robot description, xacro)
@@ -2,5 +2,4 @@
 <robot name="rosbot"
   xmlns:xacro="http://www.ros.org/wiki/xacro">
-  <xacro:property name="M_PI" value="3.1415926535897931" />
   <xacro:arg name="robot_namespace" default=""/>
   <xacro:property name="cameraSize" value="0.05"/>
@@ -286,12 +285,12 @@
   <link name="camera_depth_frame">
   </link>
-  <!-- <joint name="rplidar_joint" type="fixed">
+  <joint name="rplidar_joint" type="fixed">
     <axis xyz="0 1 0" />
     <origin xyz="0.02 0 0" rpy="0 0 3.14"/>
     <parent link="base_link"/>
     <child link="laser"/>
-  </joint> -->
+  </joint>
   <!-- rplidar Laser -->
-  <!-- <link name="laser">
+  <link name="laser">
     <collision>
       <origin xyz="0 0 0.058" rpy="1.5707 0 4.71"/>
@@ -311,56 +310,5 @@
       <inertia ixx="0" ixy="0" ixz="0" iyy="0" iyz="0" izz="0" />
     </inertial>
-  </link> -->
-<!-- Velodyne Link Stuff -->
-  <!-- <link name="laser">
-    <collision>
-      <origin xyz="0 0 0.058" rpy="1.5707 0 4.71"/>
-      <geometry>
-        <cylinder radius="0.0516" length="0.0717"/>
-      </geometry>
-    </collision>
-    <visual>
-      <origin xyz="0 0 0.058" rpy="1.5707 0 4.71"/>
-      <geometry>
-        <mesh filename="package://rosbot_description/meshes/VLP16_base_1.dae" scale="0.001 0.001 0.001" />
-      </geometry>
-    </visual>
-    <visual>
-      <origin xyz="0 0 0.058" rpy="1.5707 0 4.71"/>
-      <geometry>
-        <mesh filename="package://rosbot_description/meshes/VLP16_base_2.dae" scale="0.001 0.001 0.001" />
-      </geometry>
-    </visual>
-    <inertial>
-      <mass value="0.83"/>
-      <origin xyz="0 0 0.03585"/>
-      <inertia ixx="${(0.83 * (3.0*0.0516*0.0516 + 0.0717*0.0717)) / 12.0}" ixy="0" ixz="0"
-        iyy="${(0.83 * (3.0*0.0516*0.0516 + 0.0717*0.0717)) / 12.0}" iyz="0"
-        izz="${0.5 * 0.83 * (0.0516*0.0516)}"/>
-    </inertial>
-  </link>
-  <joint name="$laser_base_scan_joint" type="fixed" >
-    <origin xyz="0 0 0.0377" rpy="0 0 0" />
-    <parent link="laser" />
-    <child link="laser_velodyne"/>
-  </joint>
-  <link name="laser_velodyne">
-    <inertial>
-      <mass value="0.01"/>
-      <origin xyz="0 0 0"/>
-      <inertia ixx="1e-7" ixy="0" ixz="0" iyy="1e-7" iyz="0" izz="1e-7"/>
-    </inertial>
-    <visual>
-      <origin xyz="0 0 -0.0377" />
-      <geometry>
-        <mesh filename="package://rosbot_description/meshes/VLP16_scan.dae" scale="0.001 0.001 0.001" />
-      </geometry>
-    </visual>
-  </link> -->
-<!-- Velodyne Include Stuff -->
-  <xacro:include filename="$(find rosbot_description)/urdf/VLP-16-modified.urdf.xacro"/>
-  <VLP-16 parent="base_link" name="velodyne" topic="/velodyne_points" hz="10" samples="440" gpu="false">
-    <origin xyz="0.025 0 0.055" rpy="0 0 0" />
-  </VLP-16>
+  </link>
   <joint name="range_fl_joint" type="fixed">
     <axis xyz="0 1 0" />
