Commit message: Mounted velodyne lidar vertically. Created and configured quadrotor moveit package for octomap

File: lidar_interface/urdf/VLP-16-flight.urdf.xacro (robot description, xacro)
@@ -2,5 +2,5 @@
 <robot xmlns:xacro="http://www.ros.org/wiki/xacro" name="VLP-16">
   <xacro:property name="M_PI" value="3.1415926535897931" />
-  <xacro:macro name="VLP-16" params="*origin parent:=base_link name:=velodyne topic:=/velodyne_points hz:=10 lasers:=16 samples:=1875 collision_range:=0.3 min_range:=0.9 max_range:=130.0 noise:=0.008 min_angle:=-${M_PI} max_angle:=${M_PI} gpu:=false">
+  <xacro:macro name="VLP-16" params="*origin parent:=base_link name:=velodyne topic:=/velodyne_points hz:=10 lasers:=16 samples:=1875 collision_range:=0.3 min_range:=0.9 max_range:=130.0 noise:=0.008 min_angle:=-1.570796327 max_angle:=1.570796327 gpu:=false">
     <joint name="${name}_base_mount_joint" type="fixed">
       <xacro:insert_block name="origin" />

File: lidar_interface/urdf/quadrotor_velodyne.urdf.xacro (robot description, xacro)
@@ -33,5 +33,5 @@
     <xacro:include filename="$(find lidar_interface)/urdf/VLP-16-flight.urdf.xacro"/>
     <VLP-16 parent="base_link" name="velodyne" topic="/velodyne_points" hz="10" samples="440" gpu="false">
-        <origin xyz="0.0 0.0 0.07" rpy="0 0 0" />
+        <origin xyz="0.0 0.0 0.07" rpy="0 1.57079632679 0" />
     </VLP-16>
 </robot>
